File: keyboard/keyboard.kicad_sch (KiCad schematic)
At the start: 33 parts, among them J1 USB_C_Receptacle_USB2.0_16P, J2 Conn_01x04, J3 Conn_01x05, SW1 RESET_SW, SW2 BOOTTSEL_SW, U1 RP2040, U2 XC6206PxxxMR, U3 SRV05-4, U4 W25Q128JVS, Y1 Crystal_GND24

Commit message: somethignsgnfskdgb
Parts:
- added CH1, CH2, CH3, CH4: choc_v1_SW_HS, PCM_marbastlib-choc:SW_choc_v1_HS_CPG135001S30_1u, symbol PCM_marbastlib-choc:choc_v1_SW_HS_CPG135001S30
- added D1, D2, D3, D4: D_Small, symbol Device:D_Small
Connections:
- new net: CH2.2, D2.2 (A)
- new net: D3.1 (K), D4.1 (K)
- new net: CH4.2, D4.2 (A)
- new net: CH1.2, D1.2 (A)
- new net: D1.1 (K), D2.1 (K)
- new net: CH3.2, D3.2 (A)
Other:
- note removed: "3.3V Voltage Regulator"
- note removed: "Boot Selection Switch"
- note removed: "Crystal"
- note removed: "Debug Header"
- note removed: "Decoupling Capacitors"
- note removed: "ESD Protector"
- note removed: "Flash"
- note removed: "MCU"
- note removed: "Reset Switch"
- note removed: "USB-C Header"
- note removed: "USB-C Port"
- moved on the sheet: C12, R4, R5, R7, R8, R9, SW2, U1, U4
